File: electronics/fume-pcb/fume-pcb.kicad_pcb (KiCad board)
At the start: 2 copper layers, 122.8 x 87.2 mm, 1 part

Commit message: Update
Parts:
- added C1: 220uF, Capacitor_THT:CP_Radial_D6.3mm_P2.50mm, F.Cu at (179.8, 72.2)
- added C10: 22uF, Capacitor_THT:CP_Radial_D4.0mm_P2.00mm, F.Cu at (198.2, 111.2)
- added C11: 0.1uF, Capacitor_THT:C_Disc_D5.0mm_W2.5mm_P5.00mm, F.Cu at (194.2, 111.3)
- added C12: 22uF, Capacitor_THT:CP_Radial_D4.0mm_P2.00mm, F.Cu at (198.2, 119.4)
- added C13: 0.1uF, Capacitor_THT:C_Disc_D5.0mm_W2.5mm_P5.00mm, F.Cu at (194.2, 119.5)
- added C2: 22uF, Capacitor_THT:CP_Radial_D4.0mm_P2.00mm, F.Cu at (184.3, 72.2)
- added C3: 10uF, Capacitor_THT:C_Disc_D5.0mm_W2.5mm_P5.00mm, F.Cu at (181.8, 78.5)
- added C4: 1uF, Capacitor_THT:C_Disc_D5.0mm_W2.5mm_P5.00mm, F.Cu at (181.8, 82.2)
- added C5: 0.1uF, Capacitor_THT:C_Disc_D5.0mm_W2.5mm_P5.00mm, F.Cu at (181.8, 85.8)
- added C6: 1uF, Capacitor_THT:C_Disc_D5.0mm_W2.5mm_P5.00mm, F.Cu at (118.0, 87.7)
- added C7: 0.1uF, Capacitor_THT:C_Disc_D5.0mm_W2.5mm_P5.00mm, F.Cu at (118.0, 91.8)
- added C8: 22uF, Capacitor_THT:CP_Radial_D4.0mm_P2.00mm, F.Cu at (198.4, 102.8)
- added C9: 0.1uF, Capacitor_THT:C_Disc_D5.0mm_W2.5mm_P5.00mm, F.Cu at (194.2, 102.9)
- added D1: 1N5819, Diode_THT:D_DO-41_SOD81_P10.16mm_Horizontal, F.Cu at (166.2, 132.2)
- added D2: BLUE, LED_THT:LED_D5.0mm, F.Cu at (139.7, 58.2)
- added D3: RED, LED_THT:LED_D5.0mm, F.Cu at (147.7, 58.2)
- added H1: MHole, MountingHole:MountingHole_3.2mm_M3_Pad_Via, F.Cu at (91.0, 56.0)
- added H2: MHole, MountingHole:MountingHole_3.2mm_M3_Pad_Via, F.Cu at (199.0, 56.0)
- added H3: MHole, MountingHole:MountingHole_3.2mm_M3_Pad_Via, F.Cu at (199.0, 134.0)
- added H4: MHole, MountingHole:MountingHole_3.2mm_M3_Pad_Via, F.Cu at (91.0, 134.0)
- added J1: PWR Conn, Connector_BarrelJack:BarrelJack_Horizontal, F.Cu at (181.5, 66.0)
- added J2: Conn_01x02, Connector_JST:JST_XH_B2B-XH-A_1x02_P2.50mm_Vertical, F.Cu at (189.2, 119.5)
- added J3: Conn_01x03, Connector_JST:JST_XH_B3B-XH-A_1x03_P2.50mm_Vertical, F.Cu at (189.2, 111.2)
- added J4: Conn_01x04, Connector_JST:JST_XH_B4B-XH-A_1x04_P2.50mm_Vertical, F.Cu at (189.2, 103.0)
- added Q1: STP12PF06, Package_TO_SOT_THT:TO-220-3_Vertical, F.Cu at (190.0, 62.9)
- added Q2: 2N3904, Package_TO_SOT_THT:TO-92_Inline, F.Cu at (122.5, 108.2)
- added Q3: 2N3906, Package_TO_SOT_THT:TO-92_Inline, F.Cu at (146.2, 115.4)
- added Q4: 2N3904, Package_TO_SOT_THT:TO-92_Inline, F.Cu at (146.2, 109.6)
- added Q5: IRFZ44N, Package_TO_SOT_THT:TO-220-3_Vertical, F.Cu at (160.5, 129.8)
- added R1: 1k, Resistor_THT:R_Axial_DIN0207_L6.3mm_D2.5mm_P10.16mm_Horizontal, F.Cu at (108.2, 108.2)
- added R2: 4.7k, Resistor_THT:R_Axial_DIN0207_L6.3mm_D2.5mm_P10.16mm_Horizontal, F.Cu at (132.5, 95.0)
- added R3: 2.2k, Resistor_THT:R_Axial_DIN0207_L6.3mm_D2.5mm_P10.16mm_Horizontal, F.Cu at (132.5, 99.0)
- added R4: 2.2k, Resistor_THT:R_Axial_DIN0207_L6.3mm_D2.5mm_P10.16mm_Horizontal, F.Cu at (132.5, 103.1)
- added R5: 1k, Resistor_THT:R_Axial_DIN0207_L6.3mm_D2.5mm_P10.16mm_Horizontal, F.Cu at (139.8, 62.9)
- added R6: 5.1k, Resistor_THT:R_Axial_DIN0207_L6.3mm_D2.5mm_P10.16mm_Horizontal, F.Cu at (147.2, 62.9)
- added R7: 4.7k, Resistor_THT:R_Axial_DIN0207_L6.3mm_D2.5mm_P10.16mm_Horizontal, F.Cu at (132.5, 111.2)
- moved A1 5.99 mm to (125.6, 68.5), turned to -90 degrees
Connections:
- A1 pad 12: unconnected-(A1-D9-Pad12) -> /PWM_FAN
- A1 pad 13: unconnected-(A1-D10-Pad13) -> /PWM_MOS
- A1 pad 19: unconnected-(A1-A0-Pad19) -> /REF_FAN
- A1 pad 5: unconnected-(A1-D2-Pad5) -> /ENC_FAN
Other:
- board size 122.8 x 87.2 mm -> 120 x 90 mm

Commit message: Update
Parts:
- removed the D2 at (139.7, 58.2)
- removed D3: RED, LED_THT:LED_D5.0mm
- removed the R5 at (139.8, 62.9)
- added C1: 0.1uF, Capacitor_THT:C_Disc_D5.0mm_W2.5mm_P5.00mm, F.Cu at (151.4, 97.8)
- added C4: 0.1uF, Capacitor_THT:C_Disc_D5.0mm_W2.5mm_P5.00mm, F.Cu at (160.1, 104.7)
- added D1: BZW04-136, Diode_THT:D_DO-15_P10.16mm_Horizontal, F.Cu at (179.6, 70.8)
- added J5: Ref_conn, Connector_JST:JST_XH_B3B-XH-A_1x03_P2.50mm_Vertical, F.Cu at (136.4, 69.9)
- added R7: 10k, Resistor_THT:R_Axial_DIN0207_L6.3mm_D2.5mm_P10.16mm_Horizontal, F.Cu at (134.8, 97.6)
- added SW1: SW_SEL, Button_Switch_THT:SW_DIP_SPSTx02_Slide_6.7x6.64mm_W7.62mm_P2.54mm_LowProfile, F.Cu at (134.2, 84.8)
- J2: value Conn_01x02 -> 2_Wire_conn
- J3: renamed from J4; value Conn_01x04 -> 4_Wire_conn
- J4: renamed from J3; value Conn_01x03 -> 3_Wire_conn
- R6: value 5.1k -> 10k
- moved H4 49.3 mm to (138.8, 121.8)
- moved H1 46.2 mm to (137.2, 56.3)
- moved A1 42.9 mm to (162.0, 91.1), turned to 180 degrees
- moved R5 39.3 mm to (166.3, 91.1), turned to 90 degrees
- moved R6 38.7 mm to (130.3, 97.7)
- moved R1 36.5 mm to (143.1, 97.8), turned to -90 degrees
- moved C15 27.3 mm to (142.8, 80.4), turned to 90 degrees
- moved C14 25.2 mm to (142.8, 83.1), turned to -90 degrees
- moved R3 23.3 mm to (155.7, 100.7), turned to -90 degrees
- moved Q2 22.7 mm to (144.4, 113.9)
- moved R4 19.8 mm to (152.0, 106.9), turned to -90 degrees
- moved Q4 17.0 mm to (160.8, 118.2), turned to 90 degrees
- moved Q5 15.5 mm to (167.3, 116.0)
- moved Q3 15.0 mm to (160.1, 109.6), turned to -90 degrees
- moved R2 15.0 mm to (147.3, 97.8), turned to -90 degrees
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- renumbered C4 to C10, C5 to C11, C10 to C12, C11 to C13, C6 to C14, C7 to C15, C8 to C2, C12 to C3, C9 to C5, C13 to C6, C1 to C7, C2 to C8, C3 to C9, D1 to D2, R7 to R5
Connections:
- R6 pad 1: Net-(D3-K) -> /ON_PWM
Routing:
- net /VIN: track 0.00 -> 8.64 mm
- added copper zone on F.Cu, net +12V
- added copper zone on F.Cu, net +5V
Other:
- board text added: "12V"
- board text added: "ENC"
- board text added: "ENC ON"
- board text added: "Fan Conn"
- board text added: "Fan Driver"
- board text added: "GND"
- board text added: "MCU"
- board text added: "POT"
- board text added: "PWM"
- board text added: "PWM ON"
- board text added: "V1.0 Rev A"
- board text added: "VDD"
- board text added: "by Ulrik Helk"

Commit message: Update
Parts:
- removed R6, R7: 10k, Resistor_THT:R_Axial_DIN0207_L6.3mm_D2.5mm_P10.16mm_Horizontal
- added REF**: WEEE-Logo_5.6x8mm_SilkScreen, Symbol:WEEE-Logo_5.6x8mm_SilkScreen, B.Cu at (189.3, 113.3)
- moved SW1 46.2 mm to (169.9, 55.6), turned to -90 degrees
- moved H4 8.69 mm to (135.0, 114.0)
- moved H3 7.81 mm to (199.0, 114.0)
- moved Q1 6.83 mm to (191.3, 55.1)
- moved C7 6.54 mm to (179.9, 69.0)
- moved D1 5.76 mm to (185.1, 69.0)
- moved J1 5.29 mm to (184.5, 63.7)
- moved Q4 4.77 mm to (160.3, 113.5)
- moved Q3 4.72 mm to (159.5, 104.9)
- moved R4 4.41 mm to (151.7, 102.5)
- moved D2 4.31 mm to (171.6, 114.0)
- moved J5 3.73 mm to (140.1, 70.5)
- moved C12 3.72 mm to (190.3, 100.2)
- moved J2 3.72 mm to (182.0, 112.5)
- moved J3 3.72 mm to (182.0, 96.0)
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Connections:
- A1 pad 14: unconnected-(A1-D11-Pad14) -> /ON_PWM
- A1 pad 15: unconnected-(A1-D12-Pad15) -> /ON_ENC
- SW1 pad 1: +5V -> GND
- SW1 pad 2: +5V -> GND
Routing:
- net +12V: track 0.08 -> 133.8 mm
- net /PWM_FAN: track 0.00 -> 47.7 mm
- net /PWM_MOS: track 0.00 -> 46.1 mm
- net +5V: track 0.00 -> 43.1 mm, vias 0 -> 2
- net /ENC_FAN: track 0.00 -> 32.0 mm
- net /GND_FAN: track 0.39 -> 31.8 mm
- net Net-(Q2-C): track 0.00 -> 17.1 mm
- net /ON_ENC: track 0.00 -> 12.6 mm
- net Net-(Q3-C): track 0.00 -> 11.7 mm
- net Net-(Q4-B): track 0.00 -> 8.74 mm
- net /REF_FAN: track 0.00 -> 8.69 mm
- net /ON_PWM: track 0.00 -> 8.52 mm
- net Net-(Q3-B): track 0.00 -> 7.33 mm
- net Net-(Q2-B): track 0.00 -> 6.73 mm
- net /VIN: track 8.64 -> 6.84 mm
- added copper zone on B.Cu, net GND
- added copper zone on F.Cu, net GND
Other:
- board size 120 x 90 mm -> 76 x 70 mm

Commit message: Almost done with PCB
Parts:
- moved Q1 9.71 mm to (197.0, 63.0), turned to 180 degrees
- moved H1 7.88 mm to (142.9, 55.9)
- moved H4 7.88 mm to (142.9, 113.9)
- moved J5 7.02 mm to (144.8, 75.7)
- moved SW1 5.74 mm to (173.2, 60.3)
- moved Q2 4.51 mm to (149.7, 112.5)
- moved C3 4.37 mm to (194.2, 108.1), turned to 90 degrees
- moved C2 4.30 mm to (194.2, 91.6), turned to 90 degrees
- moved R5 4.01 mm to (170.0, 92.7)
- moved C12 3.95 mm to (194.2, 99.8), turned to 90 degrees
- moved C10 3.88 mm to (183.8, 78.4)
- moved C11 3.88 mm to (183.8, 81.9)
- moved C9 3.88 mm to (183.8, 74.6)
- moved R1 3.88 mm to (148.2, 97.7)
- moved R4 3.88 mm to (155.6, 102.4)
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Connections:
- A1 pad 19: /REF_FAN -> unconnected-(A1-A0-Pad19)
- A1 pad 23: unconnected-(A1-A4-Pad23) -> /REF_FAN
- J1 pad 1: GND -> /VIN
- J1 pad 2: /VIN -> GND
- J1 pad 3: (no net) -> GND
Routing:
- net /ON_ENC: track 12.6 -> 0.00 mm
- net /ON_PWM: track 8.52 -> 0.24 mm
- net +5V: track 43.1 -> 36.0 mm
- net /VIN: track 6.84 -> 13.9 mm
- net +12V: track 133.8 -> 127.1 mm
- net GND: track 0.00 -> 5.65 mm
- net /GND_FAN: track 31.8 -> 36.1 mm
- net /REF_FAN: track 8.69 -> 5.85 mm
- net /PWM_FAN: track 47.7 -> 46.5 mm
- net Net-(Q2-C): track 17.1 -> 16.1 mm
- net Net-(Q2-B): track 6.73 -> 5.72 mm
- net Net-(Q3-C): track 11.7 -> 10.8 mm
Other:
- board size 76 x 70 mm -> 68 x 70 mm
- board text added: "0"
- board text added: "1"
- board text removed: "ENC ON"
- board text removed: "PWM ON"

Commit message: PCB ORDERED
Parts:
- removed REF**: WEEE-Logo_5.6x8mm_SilkScreen, Symbol:WEEE-Logo_5.6x8mm_SilkScreen
- added G***: LOGO, 0_logo:fan_80x80mm, B.Cu at (170.0, 85.0)
- added R6: 10k, Resistor_THT:R_Axial_DIN0207_L6.3mm_D2.5mm_P10.16mm_Horizontal, F.Cu at (144.7, 107.9)
- moved SW1 7.98 mm to (170.7, 67.8), turned to 90 degrees
- moved H1 2.00 mm to (140.9, 55.9)
- moved H4 2.00 mm to (140.9, 113.9)
- moved J5 1.10 mm to (143.7, 75.7)
- moved R5 0.37 mm to (169.6, 92.8)
Connections:
- A1 pad 14: /ON_PWM -> /ON_ENC
- A1 pad 15: /ON_ENC -> /ON_PWM
Routing:
- net /ON_PWM: track 0.24 -> 9.89 mm
- net /ON_ENC: track 0.00 -> 5.94 mm
- net /PWM_MOS: track 46.1 -> 49.6 mm
- net /ENC_FAN: track 32.5 -> 30.9 mm
- net /REF_FAN: track 5.85 -> 7.17 mm
- net /PWM_FAN: track 46.5 -> 47.2 mm
- net +5V: track 36.0 -> 36.4 mm, vias 2 -> 0
- net GND: vias 0 -> 1727
Other:
- board size 68 x 70 mm -> 70 x 70 mm
- board text added: "M3 mounting pitch 58mm"
- board text added: "he1k 03/25"
