File: electronics/fume-pcb/fume-pcb.kicad_sch (KiCad schematic)
At the start: 2 parts

Commit message: Update
Parts:
- removed R1: R_Small, symbol Device:R_Small
Changed lines of the file:
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@@
-	)
-	(symbol
-		(lib_id "Device:R_Small")
-		(at 77.47 66.04 0)
-		(unit 1)
-		(exclude_from_sim no)
-		(in_bom yes)
-		(on_board yes)
-		(dnp no)
-		(fields_autoplaced yes)
-		(property "Reference" "R1"
-			(at 80.01 64.7699 0)
-			(effects
-				(font
-					(size 1.27 1.27)
-				)
-				(justify left)
-			)
-		)
-		(property "Value" "R_Small"
-			(at 80.01 67.3099 0)
-			(effects
-				(font
-					(size 1.27 1.27)
-				)
-				(justify left)
-			)
-		)
-		(property "Footprint" ""
-			(at 77.47 66.04 0)
-			(effects
-				(font
-					(size 1.27 1.27)
-				)
-				(hide yes)
-			)
-		)
-		(property "Datasheet" "~"
-			(at 77.47 66.04 0)
-			(effects
-				(font
-					(size 1.27 1.27)
-				)
-				(hide yes)
-			)
-		)
-		(property "Description" "Resistor, small symbol"
-			(at 77.47 66.04 0)
-			(effects
-				(font
-					(size 1.27 1.27)
-				)
-				(hide yes)
-			)
-		)
-		(pin "2"
-		)
-		(pin "1"
-		)
-		(instances
-			(project ""
-				(path "/c9144cb8-ec55-40f4-a57c-9e7a9024dc9f"
-					(reference "R1")
-					(unit 1)
-				)
-			)
-		)
 	)
 	(symbol

Commit message: Update
Parts:
- added C1: 220uF, Capacitor_THT:CP_Radial_D6.3mm_P2.50mm, symbol Device:C_Polarized_Small
- added C10, C12, C2, C8: 22uF, Capacitor_THT:CP_Radial_D4.0mm_P2.00mm, symbol Device:C_Polarized_Small
- added C11, C13, C5, C7, C9: 0.1uF, Capacitor_THT:C_Disc_D5.0mm_W2.5mm_P5.00mm, symbol Device:C_Small
- added C3: 10uF, Capacitor_THT:C_Disc_D5.0mm_W2.5mm_P5.00mm, symbol Device:C_Small
- added C4, C6: 1uF, Capacitor_THT:C_Disc_D5.0mm_W2.5mm_P5.00mm, symbol Device:C_Small
- added D1: 1N5819, Diode_THT:D_DO-41_SOD81_P10.16mm_Horizontal, symbol Diode:1N5819
- added D2: BLUE, LED_THT:LED_D5.0mm, symbol Device:LED
- added D3: RED, LED_THT:LED_D5.0mm, symbol Device:LED
- added H1, H2, H3, H4: MHole, MountingHole:MountingHole_3.2mm_M3_Pad_Via, symbol Mechanical:MountingHole_Pad
- added J1: PWR Conn, Connector_BarrelJack:BarrelJack_Horizontal, symbol Connector_Generic:Conn_01x02
- added J2: Conn_01x02, Connector_JST:JST_XH_B2B-XH-A_1x02_P2.50mm_Vertical, symbol Connector_Generic:Conn_01x02
- added J3: Conn_01x03, Connector_JST:JST_XH_B3B-XH-A_1x03_P2.50mm_Vertical, symbol Connector_Generic:Conn_01x03
- added J4: Conn_01x04, Connector_JST:JST_XH_B4B-XH-A_1x04_P2.50mm_Vertical, symbol Connector_Generic:Conn_01x04
- added Q1: STP12PF06, Package_TO_SOT_THT:TO-220-3_Vertical, symbol Device:Q_PMOS_GDS
- added Q2, Q4: 2N3904, Package_TO_SOT_THT:TO-92_Inline, symbol Transistor_BJT:2N3904
- added Q3: 2N3906, Package_TO_SOT_THT:TO-92_Inline, symbol Transistor_BJT:2N3906
- added Q5: IRFZ44N, Package_TO_SOT_THT:TO-220-3_Vertical, symbol Device:Q_NMOS_GDS
- added R1, R5: 1k, Resistor_THT:R_Axial_DIN0207_L6.3mm_D2.5mm_P10.16mm_Horizontal, symbol Device:R_Small
- added R2, R7: 4.7k, Resistor_THT:R_Axial_DIN0207_L6.3mm_D2.5mm_P10.16mm_Horizontal, symbol Device:R_Small
- added R3, R4: 2.2k, Resistor_THT:R_Axial_DIN0207_L6.3mm_D2.5mm_P10.16mm_Horizontal, symbol Device:R_Small
- added R6: 5.1k, Resistor_THT:R_Axial_DIN0207_L6.3mm_D2.5mm_P10.16mm_Horizontal, symbol Device:R_Small
Connections:
- net +12V: now also C1.1, C10.1, C11.1, C12.1, C13.1, C2.1, C3.1, C4.1, C5.1, C8.1, C9.1, D3.2 (A), J2.1 (Pin_1), J3.1 (Pin_1), J4.1 (Pin_1), Q1.3 (S), Q3.1 (E), R2.1
- net +5V: now also C6.1, C7.1, D2.2 (A), R7.1
- net GND: now also C1.2, C10.2, C11.2, C12.2, C13.2, C2.2, C3.2, C4.2, C5.2, C6.2, C7.2, C8.2, C9.2, D1.2 (A), H1.1, H2.1, H3.1, H4.1, J1.1 (Pin_1), Q1.1 (G), Q2.1 (E), Q4.1 (E), Q5.3 (S), R5.2, R6.2
- net PWM_FAN: now reaches A1.12 (D9)
- net PWM_FAN: now also J4.4 (Pin_4)
- net PWM_MOS: now reaches A1.13 (D10)
- net PWM_MOS: now also R1.1
- net REF_FAN: now reaches A1.19 (A0)
- net ENC_FAN: now reaches A1.5 (D2)
- net ENC_FAN: now also J3.3 (Pin_3), J4.3 (Pin_3), R7.2
- new net: D2.1 (K), R5.1
- new net: Q3.2 (B), R3.2
- new net: Q3.3 (C), Q4.3 (C), Q5.1 (G)
- new net: D3.1 (K), R6.1
- new net: Q2.3 (C), R2.2, R3.1, R4.1
- new net: Q4.2 (B), R4.2
- new net: Q2.2 (B), R1.2
- new net GND_FAN: D1.1 (K), J2.2 (Pin_2), J3.2 (Pin_2), J4.2 (Pin_2), Q5.2 (D)
- new net VIN: J1.2 (Pin_2), Q1.2 (D)
- no-connect marks 8 -> 20
Other:
- note added: "2 wire fan"
- note added: "3 wire fan"
- note added: "4 wire fan"
- note added: "ARDUINO NANO"
- note added: "CONNECTORS ETC."
- note added: "GATE DRIVER AND MOSFET"
- note added: "INDICATORS"
- note added: "MOUNTING"
- note added: "POWER"
- note added: "Reverse polarity protection"
- moved on the sheet: A1

Commit message: Update
Parts:
- removed D2: BLUE, LED_THT:LED_D5.0mm, symbol Device:LED
- removed D3: RED, LED_THT:LED_D5.0mm, symbol Device:LED
- removed R5: 1k, Resistor_THT:R_Axial_DIN0207_L6.3mm_D2.5mm_P10.16mm_Horizontal, symbol Device:R_Small
- added C1, C4: 0.1uF, Capacitor_THT:C_Disc_D5.0mm_W2.5mm_P5.00mm, symbol Device:C_Small
- added D1: BZW04-136, Diode_THT:D_DO-15_P10.16mm_Horizontal, symbol Device:D_Zener_Small
- added J5: Ref_conn, Connector_JST:JST_XH_B3B-XH-A_1x03_P2.50mm_Vertical, symbol Connector_Generic:Conn_01x03
- added R7: 10k, Resistor_THT:R_Axial_DIN0207_L6.3mm_D2.5mm_P10.16mm_Horizontal, symbol Device:R_Small
- added SW1: SW_SEL, Button_Switch_THT:SW_DIP_SPSTx02_Slide_6.7x6.64mm_W7.62mm_P2.54mm_LowProfile, symbol Switch:SW_DIP_x02
- J2: value Conn_01x02 -> 2_Wire_conn
- J3: renamed from J4; value Conn_01x04 -> 4_Wire_conn
- J4: renamed from J3; value Conn_01x03 -> 3_Wire_conn
- R6: value 5.1k -> 10k
- renumbered C4 to C10, C5 to C11, C10 to C12, C11 to C13, C6 to C14, C7 to C15, C8 to C2, C12 to C3, C9 to C5, C13 to C6, C1 to C7, C2 to C8, C3 to C9, D1 to D2, R7 to R5
Connections:
- net +12V: now also C1.1, C4.1, D1.1 (K)
- net +5V: now also J5.1 (Pin_1), SW1.1, SW1.2
- net GND: now also C1.2, C4.2, D1.2 (A), J5.3 (Pin_3), R7.2
- net REF_FAN: now also J5.2 (Pin_2)
- net ON_PWM: now reaches R6.1
- net ON_PWM: now also SW1.3
- new net ON_ENC: R7.1, SW1.4
Other:
- note removed: "INDICATORS"
- moved on the sheet: C10, C11, C12, C13, C2, C3, C5, C6, C7, C8, C9, D2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

Commit message: Update
Parts:
- removed R6, R7: 10k, Resistor_THT:R_Axial_DIN0207_L6.3mm_D2.5mm_P10.16mm_Horizontal, symbol Device:R_Small
Connections:
- net +5V: no longer SW1.1, SW1.2
- net GND: now also SW1.1, SW1.2
- net ON_ENC: now also A1.15 (D12)
- net ON_PWM: now also A1.14 (D11)
- no-connect marks 20 -> 19

Commit message: Almost done with PCB
Parts:
- removed J1: PWR Conn, Connector_BarrelJack:BarrelJack_Horizontal, symbol Connector_Generic:Conn_01x02
- added J1: PWR Conn, Connector_BarrelJack:BarrelJack_Horizontal, symbol Connector_Generic:Conn_01x03
Connections:
- net GND: now also J1.2 (Pin_2), J1.3 (Pin_3)
- net REF_FAN: now also A1.23 (A4); no longer A1.19 (A0)
- net VIN: now also J1.1 (Pin_1)
Changed lines of the file:
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@@
 	(paper "A4")
 	(junction
+		(at 30.48 34.29)
+		(diameter 0)
+		(color 0 0 0 0)
+	)
+	(junction
 		(at 49.53 71.12)
 		(diameter 0)
@@
 	)
 	(no_connect
+		(at 245.11 67.31)
+	)
+	(no_connect
 		(at 245.11 72.39)
 	)
@@
 	)
 	(no_connect
-		(at 245.11 77.47)
-	)
-	(no_connect
 		(at 219.71 69.85)
 	)
@@
 	(wire
 		(pts
-			(xy 26.67 30.48) (xy 29.21 30.48)
+			(xy 30.48 31.75) (xy 30.48 34.29)
+		)
+		(stroke
+			(width 0)
+			(type default)
+		)
+	)
+	(wire
+		(pts
+			(xy 27.94 29.21) (xy 30.48 29.21)
 		)
 		(stroke
@@
 	(wire
 		(pts
-			(xy 29.21 33.02) (xy 26.67 33.02)
+			(xy 30.48 34.29) (xy 27.94 34.29)
 		)
 		(stroke
@@
 	(wire
 		(pts
-			(xy 29.21 35.56) (xy 29.21 33.02)
+			(xy 30.48 36.83) (xy 30.48 34.29)
 		)
 		(stroke
@@
 	(wire
 		(pts
+			(xy 27.94 31.75) (xy 30.48 31.75)
+		)
+		(stroke
+			(width 0)
+			(type default)
+		)
+	)
+	(wire
+		(pts
 			(xy 76.2 68.58) (xy 76.2 71.12)
 		)
@@
 	(wire
 		(pts
-			(xy 245.11 67.31) (xy 247.65 67.31)
+			(xy 245.11 77.47) (xy 247.65 77.47)
 		)
 		(stroke
@@
 	)
 	(label "VIN"
-		(at 29.21 30.48 0)
+		(at 30.48 29.21 0)
 		(fields_autoplaced yes)
 		(effects
@@
 	)
 	(label "REF_FAN"
-		(at 247.65 67.31 0)
+		(at 247.65 77.47 0)
 		(fields_autoplaced yes)
 		(effects
@@
 	)
 	(symbol
-		(lib_id "Connector_Generic:Conn_01x02")
-		(at 21.59 33.02 180)
-		(unit 1)
-		(exclude_from_sim no)
-		(in_bom yes)
-		(on_board yes)
-		(dnp no)
-		(fields_autoplaced yes)
-		(property "Reference" "J1"
-			(at 21.59 24.13 0)
-			(effects
-				(font
-					(size 1.27 1.27)
-				)
-			)
-		)
-		(property "Value" "PWR Conn"
-			(at 21.59 26.67 0)
-			(effects
-				(font
-					(size 1.27 1.27)
-				)
-			)
-		)
-		(property "Footprint" "Connector_BarrelJack:BarrelJack_Horizontal"
-			(at 21.59 33.02 0)
-			(effects
-				(font
-					(size 1.27 1.27)
-				)
-				(hide yes)
-			)
-		)
-		(property "Datasheet" "~"
-			(at 21.59 33.02 0)
-			(effects
-				(font
-					(size 1.27 1.27)
-				)
-				(hide yes)
-			)
-		)
-		(property "Description" "Generic connector, single row, 01x02, script generated (kicad-library-utils/schlib/autogen/connector/)"
-			(at 21.59 33.02 0)
-			(effects
-				(font
-					(size 1.27 1.27)
-				)
-				(hide yes)
-			)
-		)
-		(pin "2"
-		)
-		(pin "1"
-		)
-		(instances
-			(project ""
-				(path "/c9144cb8-ec55-40f4-a57c-9e7a9024dc9f"
-					(reference "J1")
-					(unit 1)
-				)
-			)
-		)
-	)
-	(symbol
 		(lib_id "Device:C_Small")
 		(at 148.59 158.75 0)
@@
 	(symbol
 		(lib_id "power:GND")
-		(at 29.21 35.56 0)
+		(at 30.48 36.83 0)
 		(unit 1)
 		(exclude_from_sim no)
@@
 		(fields_autoplaced yes)
 		(property "Reference" "#PWR03"
-			(at 29.21 41.91 0)
+			(at 30.48 43.18 0)
 			(effects
 				(font
@@
 		)
 		(property "Value" "GND"
-			(at 29.21 40.64 0)
+			(at 30.48 41.91 0)
 			(effects
 				(font
@@
 		)
 		(property "Footprint" ""
-			(at 29.21 35.56 0)
+			(at 30.48 36.83 0)
 			(effects
 				(font
@@
 		)
 		(property "Datasheet" ""
-			(at 29.21 35.56 0)
+			(at 30.48 36.83 0)
 			(effects
 				(font
@@
 		)
 		(property "Description" "Power symbol creates a global label with name \"GND\" , ground"
-			(at 29.21 35.56 0)
+			(at 30.48 36.83 0)
 			(effects
 				(font
@@
 					(unit 1)
 				)
+			)
+		)
+	)
+	(symbol
+		(lib_id "Connector_Generic:Conn_01x03")
+		(at 22.86 31.75 0)
+		(mirror y)
+		(unit 1)
+		(exclude_from_sim no)
+		(in_bom yes)
+		(on_board yes)
+		(dnp no)
+		(property "Reference" "J1"
+			(at 22.86 26.162 0)
+			(effects
+				(font
+					(size 1.27 1.27)
+				)
+			)
+		)
+		(property "Value" "PWR Conn"
+			(at 22.86 23.622 0)
+			(effects
+				(font
+					(size 1.27 1.27)
+				)
+			)
+		)
+		(property "Footprint" "Connector_BarrelJack:BarrelJack_Horizontal"
+			(at 22.86 31.75 0)
+			(effects
+				(font
+					(size 1.27 1.27)
+				)
+				(hide yes)
+			)
+		)
+		(property "Datasheet" "~"
+			(at 22.86 31.75 0)
+			(effects
+				(font
+					(size 1.27 1.27)
+				)
+				(hide yes)
+			)
+		)
+		(property "Description" "Generic connector, single row, 01x03, script generated (kicad-library-utils/schlib/autogen/connector/)"
+			(at 22.86 31.75 0)
+			(effects
+				(font
+					(size 1.27 1.27)
+				)
+				(hide yes)
+			)
+		)
+		(pin "1"
+		)
+		(pin "2"
+		)
+		(pin "3"
+		)
+		(instances
+			(project ""
+				(path "/c9144cb8-ec55-40f4-a57c-9e7a9024dc9f"
+					(reference "J1")
+					(unit 1)
+				)

Commit message: PCB ORDERED
Parts:
- added R6: 10k, Resistor_THT:R_Axial_DIN0207_L6.3mm_D2.5mm_P10.16mm_Horizontal, symbol Device:R_Small
Connections:
- net GND: now also R6.1
- net ON_ENC: now also A1.14 (D11); no longer A1.15 (D12)
- net ON_PWM: now also A1.15 (D12); no longer A1.14 (D11)
- net PWM_MOS: now also R6.2
Other:
- moved on the sheet: C1, C4, D2, Q2, Q3, Q4, Q5, R1, R2, R3, R4
